Commit message: feat: data collections, update urdf, env

File: genesis_ILDP/assets/roboticArms/urdf/plane.urdf (robot description, URDF)
Before this commit: robot plane_with_cube_marker, 2 links, 1 joints
Joints:
- joint marker_joint: origin xyz=0.5 0.5 0.01 rpy=0 0 0 -> xyz=0.5 0.5 0.03 rpy=0 0 0

Commit message: modified:   genesis_ILDP/assets/roboticArms/urdf/cube.urdf 	modified:   genesis_ILDP/assets/roboticArms/urdf/plane.urdf 	modified:   genesis_ILDP/env/pushT_env.py 	modified:   genesis_ILDP/scipt/img/PushTEnv-0.jpg 	modified:   genesis_ILDP/scipt/img/PushTEnv-1.jpg 	modified:   genesis_ILDP/scipt/img/PushTEnv-2.jpg 	modified:   genesis_ILDP/scipt/img/PushTEnv-3.jpg 	modified:   genesis_ILDP/scipt/img/PushTEnv-4.jpg 	modified:   genesis_ILDP/scipt/img/PushTEnv-5.jpg 	modified:   genesis_ILDP/scipt/img/PushTEnv-6.jpg 	modified:   genesis_ILDP/scipt/img/PushTEnv-7.jpg 	modified:   genesis_ILDP/scipt/img/PushTEnv-8.jpg 	modified:   genesis_ILDP/scipt/img/PushTEnv-9.jpg

File: genesis_ILDP/assets/roboticArms/urdf/plane.urdf (robot description, URDF)
Before this commit: robot plane_with_cube_marker, 2 links, 1 joints
Links:
- added link cube, mass 0.2; collision box size=0.1 0.1 0.1; visual box size=0.1 0.1 0.1
- link marker: geometry visual box size=0.11 0.11 0.11
Joints:
- added joint cube_plane_joint: type floating, parent plane, child cube, origin xyz=0 0 0.1 rpy=0 0 0
- joint marker_joint: origin xyz=0.5 0.5 0.01 rpy=0 0 0 -> xyz=-0.5 -0.5 0.1 rpy=0 0 0

Commit message: feat. enable resetting marker pos, improve project structure

File: genesis_ILDP/assets/roboticArms/urdf/plane.urdf (robot description, URDF)
Before this commit: robot plane_with_cube_marker, 2 links, 1 joints
Links:
- added link world
- link marker: mass None -> 100
- link plane: mass 1 -> 10000; geometry collision box size=200 200 10; visual box size=200 200 10
Joints:
- added joint plane_joint: type fixed, parent world, child plane, origin xyz=0 0.0 -5.0 rpy=0 0 0
- joint marker_joint: origin xyz=0.5 0.5 0.03 rpy=0 0 0 -> xyz=0.5 0.0 0.04 rpy=0 0 0; parent plane -> world; type fixed -> floating

Commit message: feat: Change object and marker into T shape; Update: Project Structure[add reference package(mainly for testing policy), mimic its project structure and do some refinements], reminder: this version could be messy, including some copied files needed to be marked

File: genesis_ILDP/assets/roboticArms/urdf/plane.urdf (robot description, URDF)
Before this commit: robot plane_with_cube_marker, 3 links, 2 joints
Links:
- added link cubeHL, mass 0.2; visual box size=0.06 0.1 0.001
- added link cubeHR, mass 0.2; visual box size=0.06 0.1 0.001
- added link cubeV1, mass 0.2; visual box size=0.1 0.06 0.001
- added link cubeV2, mass 0.2; visual box size=0.1 0.06 0.001
- link marker: mass 100 -> None; geometry 
Joints:
- added joint Horizontal_joint_bottom1: type fixed, parent marker, child cubeV1, origin xyz=-0.08 0 0 rpy=0 0 0
- added joint Horizontal_joint_bottom2: type fixed, parent cubeV1, child cubeV2, origin xyz=-0.1 0 0 rpy=0 0 0
- added joint Horizontal_joint_left: type fixed, parent marker, child cubeHL, origin xyz=0 -0.05 0 rpy=0 0 0
- added joint Horizontal_joint_right: type fixed, parent marker, child cubeHR, origin xyz=0 0.05 0 rpy=0 0 0
- joint marker_joint: origin xyz=0.5 0.0 0.04 rpy=0 0 0 -> xyz=0 0 0.1 rpy=0 0 0
