Commit message: feat: add done condtion, reward function, pose capture... in pushT_env.py, write a simple server and client code for collecting demo data(env_server should run on server ! try to build connections)

File: genesis_ILDP/assets/roboticArms/urdf/TCube.urdf (robot description, URDF)
Before this commit: robot TCube, 6 links, 5 joints
Joints:
- joint Horizontal_joint_bottom1: origin xyz=-0.08 0 0 rpy=0 0 0 -> xyz=0.08 0 0 rpy=0 0 0
- joint Horizontal_joint_bottom2: origin xyz=-0.1 0 0 rpy=0 0 0 -> xyz=0.1 0 0 rpy=0 0 0

File: genesis_ILDP/assets/roboticArms/urdf/plane.urdf (robot description, URDF)
Before this commit: robot plane_with_Tcube_marker, 7 links, 6 joints
Joints:
- joint Horizontal_joint_bottom1: origin xyz=-0.08 0 0 rpy=0 0 0 -> xyz=0.08 0 0 rpy=0 0 0
- joint Horizontal_joint_bottom2: origin xyz=-0.1 0 0 rpy=0 0 0 -> xyz=0.1 0 0 rpy=0 0 0
